Commit message: Apply the measured calibration the 2026-08-16 sync left behind
The workspace measured all three of these between 08-10 and 08-15, but only
the 10 Hz image-stream change reached this repo. Everything else stayed on
factory or placeholder values here.

  camera_d435.yaml       Kalibr pinhole-radtan, 1637/1879 frames, 0.221 px
                         reprojection. The firmware reports zero distortion;
                         the lens really has k1 +0.108 / k2 -0.237, and cy is
                         6.4 px off factory (two recordings agreed to 0.1 px).
  bunker_d435.urdf.xacro VLP-16 moved to the front-left vent 2026-07-30
                         (0.229, 0.276, 0.0371). The value here was the 07-29
                         temporary placement and disagreed with frames.yaml.
  slam.launch.py         imu_link is no longer a placeholder at the chassis
                         origin: measured mount, and a -90 deg yaw because the
                         vectornav driver publishes RFU, not FLU.

calib/ carries the evidence: 24 h Allan deviation for the VN-100 (imu.yaml,
acceleration.png, gyro.png) and the Kalibr intrinsic and camera-IMU reports.
tools/calib_to_yaml.py converts a Kalibr camchain into the fast_livo form.

File: bunker_description/urdf/bunker_d435.urdf.xacro (robot description, xacro)
@@ -1037,13 +1037,15 @@
   -->
   <!-- ================== Velodyne VLP-16 ================== -->
-  <!-- 2026-07-29: 실측 반영. chassis→velodyne(스캔 프레임)이 x=0.240, z=0.0943 이고
-       VLP-16 매크로 내부의 base_scan_joint 0.0377 을 빼서 앞단에 0.0566 을 넣는다.
-       (이전 값 [0, 0, 0.197] 은 라이다 원위치 기준의 옛 URDF 값이었다.
-        WORKLOG 의 "VLP-16 이 임시로 옆에 내려와 있음" 상태를 반영한 것이 현재 값)
+  <!-- 2026-07-30 재배치: 라이다를 앞-왼쪽 환풍구 위에 직치 (중심선 아님, 왼쪽 27.6cm).
+       bunker_tf/config/frames.yaml 값: velodyne_base_link (0.229, 0.276, 0.0371),
+       스캔 프레임은 매크로 내부 base_scan_joint 0.0377 이 더해져 z=0.0748 이 된다.
+       (2026-08-09 확인: 이전 값 [0.240, 0, 0.0566] 은 07-29 임시 배치 기준이라
+        frames.yaml 과 어긋나 있었다. 사용자 확인 후 갱신.)
+       ★ 이 값을 바꾸면 velodyne16_vn100.yaml 의 extrinsic_T / Pcl 도 같이 갱신할 것.
        ★ bunker_tf/config/frames.yaml 과 반드시 같은 값이어야 한다. -->
   <!-- 스캔 프레임 링크명은 velodyne 드라이버 기본 frame_id인 'velodyne'과 일치시킴. -->
   <xacro:include filename="$(find velodyne_description)/urdf/VLP-16.urdf.xacro" />
   <xacro:VLP-16 parent="chassis" name="velodyne" topic="/velodyne_points">
-    <origin xyz="0.240 0 0.0566" rpy="0 0 0" />
+    <origin xyz="0.229 0.276 0.0371" rpy="0 0 0" />
   </xacro:VLP-16>
 </robot>

Commit message: Give imu_link a joint in the URDF and stop publishing it three times
The vectornav went onto the rig after bunker_d435.urdf.xacro was written, so the
URDF ended up with the mount recorded as a comment and no link to go with it.
slam.launch.py filled the gap with a static_transform_publisher, view.launch.py
published the same chassis->imu_link edge again with no arguments at all -- that
is, identity -- and odom_tf_relay carries the same numbers a third time as
parameters. Three sources for one measurement, one of them already wrong.

imu_joint now sits in the URDF next to camera_joint and the VLP-16 include,
where the other two mounts already live: [0.380, 0, 0.0371] from chassis, yaw
-90. Same x as the camera mount screw, same z as velodyne_base_link on the top
plate, and the camera 10 cm above it, which is what the 2026-07-30 measurement
note in that file says. The yaw is not the mount being rotated; imu_link is RFU
because the vectornav driver comes up with use_enu=true, and extrinsic_R in
velodyne16_vn100.yaml holds the same rotation.

With that in place slam.launch.py loses tf_nodes and the static_tf helper
entirely, and view.launch.py loses the duplicate. /tf_static now comes from
robot_state_publisher alone, and tf2_echo chassis imu_link reports
[0.380, 0.000, 0.037] at -90.000 degrees -- the same transform the deleted node
was publishing.

odom_tf_relay still holds the numbers separately because it reads odometry
rather than TF, so it cannot look them up; its comment now names imu_joint as
the thing to keep in step. view.launch.py keeps its map->camera_init publisher,
which is a deliberate identity alias for bags recorded before the frame rename,
not a mount.

File: bunker_description/urdf/bunker_d435.urdf.xacro (robot description, xacro)
@@ -1036,4 +1036,33 @@
   </xacro:innoviz_one>
   -->
+  <!-- ================== VectorNav VN-100 ================== -->
+  <!-- 2026-08-27: 여태 URDF 에 없어서 slam.launch.py 가 static_transform_publisher
+       로 따로 발행하고 있었다. 벡터나브를 리그에 나중에 얹으면서 URDF 에는 실측
+       주석(999 줄)만 남고 링크는 안 만들어진 상태였다. 같은 치수가 launch 파일과
+       view.launch.py 에 흩어져 있었고 그중 하나는 이미 (0,0,0) 으로 틀려 있었다.
+       chassis 기준 [0.380, 0, 0.0371] = 앞끝-15cm, 상판 위. 카메라 마운트 나사와
+       x 가 같고(0.380), 카메라는 여기서 10cm 위다. 999 줄 실측 그대로다.
+       z 0.0371 은 velodyne_base_link 와 같은 상판 높이.
+       ★ rpy 의 yaw -90도는 마운트가 돌아가 있어서가 아니라 imu_link 축이 RFU 라서다.
+         vectornav 드라이버가 use_enu=true 로 기동하기 때문이고, ROS 표준 FLU 가
+         아니다. velodyne16_vn100.yaml 의 extrinsic_R 이 같은 회전을 담고 있다.
+       ★ 이 값을 바꾸면 slam.launch.py 의 odom_tf_relay imu_in_base_xyz 도 같이
+         갱신할 것 (거기 값은 base_link 기준이라 z 에 chassis_joint 0.332 를 더한다).
+       ★ bunker_tf/config/frames.yaml 과 반드시 같은 값이어야 한다. -->
+  <joint name="imu_joint" type="fixed">
+    <origin xyz="0.380 0 0.0371" rpy="0 0 ${-pi/2}" />
+    <parent link="chassis" />
+    <child link="imu_link" />
+  </joint>
+  <link name="imu_link">
+    <visual>
+      <geometry>
+        <box size="0.036 0.033 0.009" />
+      </geometry>
+      <material name="vn100_black">
+        <color rgba="0.15 0.15 0.15 1" />
+      </material>
+    </visual>
+  </link>
   <!-- ================== Velodyne VLP-16 ================== -->
   <!-- 2026-07-30 재배치: 라이다를 앞-왼쪽 환풍구 위에 직치 (중심선 아님, 왼쪽 27.6cm).
